File: conformal-antennas/_autosave-conformal-antennas.kicad_pcb (KiCad board)
At the start: 2 copper layers, 1 part, among them J1 Conn_Coaxial

Commit message: adding the patch??
Routing:
- net (no net): track 0.50 -> 0.00 mm
Changed lines of the file:
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@@
 		)
-	)
-	(segment
-		(start 247.5 119)
-		(end 247.5 118.5)
-		(width 0.2)
-		(layer "F.Cu")
-		(net 0)
 	)
 	(zone
