File: conformal-antennas/conformal-antennas.kicad_sch (KiCad schematic)
At the start: 1 part, among them J1 Conn_Coaxial

Commit message: changed coaxial connector to edge mount
Parts:
- J1: footprint iclr:Molex_Nano-Fit_105313-xx02_1x02_P2.50mm_Horizontal -> Connector_Coaxial:SMA_Amphenol_132289_EdgeMount
Changed lines of the file:
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@@
 			)
 		)
-		(property "Footprint" "iclr:Molex_Nano-Fit_105313-xx02_1x02_P2.50mm_Horizontal"
+		(property "Footprint" "Connector_Coaxial:SMA_Amphenol_132289_EdgeMount"
 			(at 91.44 87.63 0)
 			(effects
